Commit message: fixed angular turning

File: urdf/components.urdf.xacro (robot description, xacro)
@@ -92,9 +92,16 @@
     <gazebo reference="${prefix}/${location_prefix}_wheel_link">
             <material>Gazebo/Black</material>
-            <mu1>100.0</mu1>
+            <!--mu1>100.0</mu1>
             <mu2>100.0</mu2>
             <kp value="1000000.0.0" />
-            <kd value="1.0" />
-            <!--fdir1 value="1 0 0"/-->
+            <kd value="1.0" /-->
+            <kp>10000000.0</kp>
+            <kd>100.0</kd>
+            <mu1>0.01</mu1>
+            <mu2>0.01</mu2>
+            <fdir1>1 1 0</fdir1>
+            <minDepth>0.00</minDepth>
+            <maxVel>2.0</maxVel>
+            <implicitSpringDamper>0</implicitSpringDamper>
     </gazebo>
     <link name="${prefix}/${location_prefix}_wheel_ver_link">
@@ -146,5 +153,5 @@
         <actuator name="${prefix}/${location_prefix}Motor">
             <hardwareInterface>VelocityJointInterface</hardwareInterface>
-            <mechanicalReduction>10</mechanicalReduction>
+            <mechanicalReduction>1</mechanicalReduction>
         </actuator>
     </transmission>
@@ -156,4 +163,5 @@
             <material name="soft_black"/>
             <geometry>
+                <!--sphere radius="${caster_wheels_radius}"/-->
                 <cylinder radius="${caster_wheels_radius}" length="${caster_wheels_length}"/>
             </geometry>
@@ -162,4 +170,5 @@
             <origin xyz="0 0 0" rpy="${math_pi/2} 0 0"/>
             <geometry>
+                <!--sphere radius="${caster_wheels_radius}"/-->
                 <cylinder radius="${caster_wheels_radius}" length="${caster_wheels_length}"/>
             </geometry>
@@ -174,4 +183,7 @@
             </physics>
         </internial>
+        <!--xacro:sphere_inertial radius="${caster_wheels_radius}" mass="${caster_wheels_mass}">
+            <origin xyz="0 0 0" rpy="0 0 0"/>
+        </xacro:sphere_inertial-->
         <xacro:cylinder_inertial radius="${caster_wheels_radius}" length="${caster_wheels_length}" mass="${caster_wheels_mass}">
             <origin xyz="0 0 0" rpy="${math_pi/2} 0 0"/>
@@ -180,9 +192,16 @@
     <gazebo reference="${prefix}/${d_location_prefix}_${r_location_prefix}_caster_wheel_link">
             <material>Gazebo/Black</material>
-            <mu1>100.0</mu1>
+            <!--mu1>100.0</mu1>
             <mu2>100.0</mu2>
             <kp value="1000000.0.0" />
-            <kd value="1.0" />
-            <!--fdir1 value="1 0 0"/-->
+            <kd value="1.0" /-->
+            <kp>10000000.0</kp>
+            <kd>100.0</kd>
+            <mu1>0.01</mu1>
+            <mu2>0.01</mu2>
+            <fdir1>1 1 0</fdir1>
+            <minDepth>0.00</minDepth>
+            <maxVel>2.0</maxVel>
+            <implicitSpringDamper>0</implicitSpringDamper>
     </gazebo>
     <link name="${prefix}/${d_location_prefix}_${r_location_prefix}_caster_wheel_ver_link">

File: urdf/definations.urdf.xacro (robot description, xacro)
@@ -5,5 +5,5 @@
         <!-- BASE -->
         <xacro:property name="base_link_w" value="0.3"/>
-        <xacro:property name="base_link_l" value="0.5"/>
+        <xacro:property name="base_link_l" value="0.3"/>
         <xacro:property name="base_link_h" value="0.2"/>
         <xacro:property name="base_link_mass" value="20.0"/>
@@ -14,10 +14,10 @@
         <xacro:property name="wheels_radius" value="0.05"/>
         <xacro:property name="wheels_length" value="0.0025"/>
-        <xacro:property name="wheels_mass" value="5.0"/>
+        <xacro:property name="wheels_mass" value="1.0"/>
         <!-- CASTER WHEEL -->
         <xacro:property name="caster_wheels_radius" value="0.025"/>
         <xacro:property name="caster_wheels_length" value="0.00125"/>
-        <xacro:property name="caster_wheels_mass" value="2.5"/>
+        <xacro:property name="caster_wheels_mass" value="0.05"/>
         <xacro:property name="effort" value="500.0"/>
-        <xacro:property name="velocity" value="100.0"/>
+        <xacro:property name="velocity" value="500.0"/>
 </robot>

Commit message: created new launch files & fixed robot wheel slipped bugs

File: urdf/components.urdf.xacro (robot description, xacro)
@@ -1,7 +1,5 @@
 <?xml version="1.0"?>
 <robot xmlns:xacro="http://www.ros.org/wiki/xacro" name="oav_components">
-    <xacro:include filename="$(find oav_description)/urdf/inertial.urdf.xacro" />
-    <xacro:include filename="$(find oav_description)/urdf/definations.urdf.xacro" />
-    <xacro:include filename="$(find oav_description)/urdf/materials.urdf.xacro" />
+    <xacro:include filename="$(find oav_description)/urdf/neshLid.urdf.xacro" />
 <xacro:macro name="base_footprint" params="prefix">
     <link name="${prefix}/base_footprint"/>
@@ -39,5 +37,5 @@
             <material>Gazebo/White</material>
     </gazebo>
-    <link name="${prefix}/base_link_turtle">
+    <!--link name="${prefix}/base_link_turtle">
         <visual>
             <origin xyz="0 0 0" rpy="0 0 ${math_pi/3}"/>
@@ -50,5 +48,5 @@
     <gazebo reference="${prefix}/base_link_turtle">
             <material>Gazebo/Green</material>
-    </gazebo>
+    </gazebo-->
     <joint name="${prefix}/base_joint" type="fixed">
         <parent link="${prefix}/base_footprint"/>
@@ -56,9 +54,9 @@
         <origin xyz="0 0 ${wheels_radius+base_link_h/2}" rpy="0 0 0"/>
     </joint>
-    <joint name="${prefix}/base_joint_turtle" type="fixed">
+    <!--joint name="${prefix}/base_joint_turtle" type="fixed">
         <parent link="${prefix}/base_link"/>
         <child link="${prefix}/base_link_turtle"/>
-        <origin xyz="${(base_link_l/2) +(turtle_link_radius)} 0 ${(base_link_h/2)+ (turtle_link_length/2)}" rpy="0 0 0"/>
-    </joint>
+        <origin xyz="${ -(turtle_link_radius)} 0 ${(base_link_h/2)+ (turtle_link_length*3/4)}" rpy="0 -0.15 0"/>
+    </joint-->
 </xacro:macro>
 <xacro:macro name="wheel_links" params="prefix location_prefix">
@@ -77,5 +75,5 @@
             </geometry>
         </collision>
-        <internial>
+        <!--internial>
             <physics type="ode">
                 <gravity xyz="0 0 -9.8"/>
@@ -85,5 +83,5 @@
                 </ode>
             </physics>
-        </internial>
+        </internial-->
         <xacro:cylinder_inertial radius="${wheels_radius}" length="${wheels_length}" mass="${wheels_mass}">
             <origin xyz="0 0 0" rpy="${math_pi/2} 0 0"/>
@@ -92,16 +90,18 @@
     <gazebo reference="${prefix}/${location_prefix}_wheel_link">
             <material>Gazebo/Black</material>
-            <!--mu1>100.0</mu1>
-            <mu2>100.0</mu2>
-            <kp value="1000000.0.0" />
-            <kd value="1.0" /-->
+             <mu1 value="200.0"/>
+             <mu2 value="200.0"/>
+            <kp value="10000000.0" />
+            <kd value="1.0" />
+            <!--
+            <material>Gazebo/Black</material>
             <kp>10000000.0</kp>
             <kd>100.0</kd>
-            <mu1>0.01</mu1>
-            <mu2>0.01</mu2>
+            <mu1>10.0</mu1>
+            <mu2>10.0</mu2>
             <fdir1>1 1 0</fdir1>
-            <minDepth>0.00</minDepth>
-            <maxVel>2.0</maxVel>
-            <implicitSpringDamper>0</implicitSpringDamper>
+            <minDepth>0.01</minDepth>
+           <implicitSpringDamper>0</implicitSpringDamper>
+            -->
     </gazebo>
     <link name="${prefix}/${location_prefix}_wheel_ver_link">
@@ -136,5 +136,6 @@
     <joint name="${prefix}/${location_prefix}_wheel_joint" type="continuous">
         <axis xyz="0 1 0" rpy="0 0 0" />
-        <limit effort="${effort}" velocity="${velocity}"/>
+        <calibration rising="0.0"/>
+        <dynamics damping="0.0" friction="0.0"/>
         <parent link="${prefix}/base_link"/>
         <child link="${prefix}/${location_prefix}_wheel_link"/>
@@ -160,19 +161,19 @@
     <link name="${prefix}/${d_location_prefix}_${r_location_prefix}_caster_wheel_link">
         <visual>
-            <origin xyz="0 0 0" rpy="${math_pi/2} 0 0"/>
+            <origin xyz="0 0 0" rpy="0 0 0"/>
             <material name="soft_black"/>
             <geometry>
-                <!--sphere radius="${caster_wheels_radius}"/-->
-                <cylinder radius="${caster_wheels_radius}" length="${caster_wheels_length}"/>
+                <sphere radius="${caster_wheels_radius}"/>
+                <!--cylinder radius="${caster_wheels_radius}" length="${caster_wheels_length}"/-->
             </geometry>
         </visual>
         <collision>
-            <origin xyz="0 0 0" rpy="${math_pi/2} 0 0"/>
-            <geometry>
-                <!--sphere radius="${caster_wheels_radius}"/-->
-                <cylinder radius="${caster_wheels_radius}" length="${caster_wheels_length}"/>
+            <origin xyz="0 0 0" rpy="0 0 0"/>
+            <geometry>
+                <sphere radius="${caster_wheels_radius}"/>
+                <!--cylinder radius="${caster_wheels_radius}" length="${caster_wheels_length}"/-->
             </geometry>
         </collision>
-        <internial>
+        <!--internial>
             <physics type="ode">
                 <gravity xyz="0 0 -9.8"/>
@@ -182,28 +183,20 @@
                 </ode>
             </physics>
-        </internial>
-        <!--xacro:sphere_inertial radius="${caster_wheels_radius}" mass="${caster_wheels_mass}">
-            <origin xyz="0 0 0" rpy="0 0 0"/>
-        </xacro:sphere_inertial-->
-        <xacro:cylinder_inertial radius="${caster_wheels_radius}" length="${caster_wheels_length}" mass="${caster_wheels_mass}">
-            <origin xyz="0 0 0" rpy="${math_pi/2} 0 0"/>
-        </xacro:cylinder_inertial>
+        </internial-->
+        <xacro:sphere_inertial radius="${caster_wheels_radius}" mass="${caster_wheels_mass}">
+            <origin xyz="0 0 0" rpy="0 0 0"/>
+        </xacro:sphere_inertial>
+        <!--xacro:cylinder_inertial radius="${caster_wheels_radius}" length="${caster_wheels_length}" mass="${caster_wheels_mass}">
+            <origin xyz="0 0 0" rpy="${math_pi/2} 0 0"/>
+        </xacro:cylinder_inertial-->
     </link>
     <gazebo reference="${prefix}/${d_location_prefix}_${r_location_prefix}_caster_wheel_link">
             <material>Gazebo/Black</material>
-            <!--mu1>100.0</mu1>
-            <mu2>100.0</mu2>
-            <kp value="1000000.0.0" />
-            <kd value="1.0" /-->
-            <kp>10000000.0</kp>
-            <kd>100.0</kd>
-            <mu1>0.01</mu1>
-            <mu2>0.01</mu2>
-            <fdir1>1 1 0</fdir1>
-            <minDepth>0.00</minDepth>
-            <maxVel>2.0</maxVel>
-            <implicitSpringDamper>0</implicitSpringDamper>
-    </gazebo>
-    <link name="${prefix}/${d_location_prefix}_${r_location_prefix}_caster_wheel_ver_link">
+            <mu1 value="0.2"/>
+            <mu2 value="0.1"/>
+            <kp value="10000000.0" />
+            <kd value="1.0" />
+    </gazebo>
+    <!--link name="${prefix}/${d_location_prefix}_${r_location_prefix}_caster_wheel_ver_link">
         <visual>
             <origin xyz="0 0 0" rpy="0 0 ${math_pi/2}"/>
@@ -230,5 +223,5 @@
             <origin xyz="0 ${-((caster_wheels_length/2)+(caster_wheels_length/16))} 0" rpy="0 0 0"/>
         </joint>
-    </xacro:unless>
+    </xacro:unless-->
 </xacro:macro>
 <xacro:macro name="caster_wheel" params="prefix r_location_prefix d_location_prefix">
@@ -236,6 +229,6 @@
     <xacro:if value="${d_location_prefix == 'front'}">
         <joint name="${prefix}/${d_location_prefix}_${r_location_prefix}_caster_wheel_joint" type="continuous">
-            <axis xyz="0 1 0" rpy="0 0 0" />
-            <limit effort="${effort}" velocity="${velocity}"/>
+           <joint_properties damping="0.0" friction="0.0"/>
+            <axis xyz="1 1 1" rpy="0 0 0" />
             <parent link="${prefix}/base_link"/>
             <child link="${prefix}/${d_location_prefix}_${r_location_prefix}_caster_wheel_link"/>
@@ -250,6 +243,6 @@
     <xacro:unless value="${d_location_prefix == 'front'}">
         <joint name="${prefix}/${d_location_prefix}_${r_location_prefix}_caster_wheel_joint" type="continuous">
-            <axis xyz="0 1 0" rpy="0 0 0" />
-            <limit effort="${effort}" velocity="${velocity}"/>
+           <joint_properties damping="0.01" friction="1.0"/>
+            <axis xyz="1 1 1" rpy="0 0 0" />
             <parent link="${prefix}/base_link"/>
             <child link="${prefix}/${d_location_prefix}_${r_location_prefix}_caster_wheel_link"/>

File: urdf/definations.urdf.xacro (robot description, xacro)
@@ -1,4 +1,4 @@
 <?xml version="1.0"?>
-<robot xmlns:xacro="http://www.ros.org/wiki/xacro" name="oav_components">
+<robot xmlns:xacro="http://www.ros.org/wiki/xacro" name="oav_definations">
         <!-- MATH -->
         <xacro:property name="math_pi" value="3.1415" />
@@ -6,6 +6,6 @@
         <xacro:property name="base_link_w" value="0.3"/>
         <xacro:property name="base_link_l" value="0.3"/>
-        <xacro:property name="base_link_h" value="0.2"/>
-        <xacro:property name="base_link_mass" value="20.0"/>
+        <xacro:property name="base_link_h" value="0.1"/>
+        <xacro:property name="base_link_mass" value="50.0"/>
         <!-- TURTLE -->
         <xacro:property name="turtle_link_length" value="0.03125"/>
@@ -14,11 +14,17 @@
         <xacro:property name="wheels_radius" value="0.05"/>
         <xacro:property name="wheels_length" value="0.0025"/>
-        <xacro:property name="wheels_mass" value="2.0"/>
+        <xacro:property name="wheels_mass" value="2.5"/>
         <!-- CASTER WHEEL -->
         <xacro:property name="caster_wheels_radius" value="0.025"/>
-        <!--xacro:property name="caster_wheels_length" value="0.00125"/-->
         <xacro:property name="caster_wheels_length" value="0.0025"/>
-        <xacro:property name="caster_wheels_mass" value="0.1"/>
-        <xacro:property name="effort" value="500.0"/>
-        <xacro:property name="velocity" value="500.0"/>
+        <xacro:property name="caster_wheels_mass" value="1.0"/>
+        <xacro:property name="effort" value="0.0001"/>
+        <xacro:property name="velocity" value="0.0"/>
+        <xacro:property name="neshLid_v1_base_w" value="0.06"/>
+        <xacro:property name="neshLid_v1_base_l" value="0.06"/>
+        <xacro:property name="neshLid_v1_base_h" value="0.03"/>
+        <xacro:property name="neshLid_v1_base_mass" value="0.01"/>
+        <xacro:property name="neshLid_v1_scanner_length" value="0.03"/>
+        <xacro:property name="neshLid_v1_scanner_radius" value="0.02"/>
+        <xacro:property name="neshLid_v1_base_mass" value="0.005"/>
 </robot>

File: urdf/materials.urdf.xacro (robot description, xacro)
@@ -1,4 +1,4 @@
 <?xml version="1.0"?>
-<robot xmlns:xacro="http://www.ros.org/wiki/xacro" name="oav_components">
+<robot xmlns:xacro="http://www.ros.org/wiki/xacro" name="oav_materials">
     <material name="white">
         <color rgba="1.0 1.0 1.0 1.0"/>

File: urdf/oav_v1.urdf.xacro (robot description, xacro)
@@ -6,4 +6,5 @@
     <xacro:include filename="$(find oav_description)/urdf/definations.urdf.xacro" />
     <xacro:base prefix="${PREFIX}"/>
+    <xacro:neshLid_v1 prefix="${PREFIX}" parrent="base_link" x="0" y="0" z="${base_link_h/2}"/>
     <xacro:wheel prefix="${PREFIX}" location_prefix="right"/>
     <xacro:wheel prefix="${PREFIX}" location_prefix="left"/>
